File: PCB/test macropad 1.kicad_pcb (KiCad board)
At the start: 2 copper layers, 98.9 x 42 mm, 11 parts, among them J1 Oled Isplay 0.91inch 128x32, SW1 SW_Push, SW2 RotaryEncoder_Switch, SW4 SW_Push, SW6 SW_Push, SW8 SW_Push, SW9 SW_Push, U1 XIAO-RP2040-DIP

Commit message: finally finished
Connections:
- SW2 pad S2: Net-(U1-GPIO3/MOSI) -> GND
Routing:
- net Net-(U1-GPIO3/MOSI): track 32.7 -> 14.4 mm
- net GND: track 339.5 -> 355.0 mm
Changed lines of the file:
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@@
 	(net 12 "Net-(U1-GPIO0{slash}TX)")
 	(net 13 "Net-(U1-GPIO28{slash}ADC2{slash}A2)")
-	(net 14 "unconnected-(U1-3V3-Pad12)")
-	(net 15 "Net-(J1-Pin_4)")
-	(net 16 "Net-(J1-Pin_3)")
+	(net 14 "Net-(J1-Pin_4)")
+	(net 15 "Net-(J1-Pin_3)")
+	(net 16 "unconnected-(U1-3V3-Pad12)_1")
 	(footprint "logo 1 random:logo"
 		(layer "F.Cu")
@@
 			(layers "F.Cu" "F.Mask")
 			(roundrect_rratio 0.1)
-			(net 15 "Net-(J1-Pin_4)")
+			(net 14 "Net-(J1-Pin_4)")
 			(pinfunction "GPIO6/SDA")
 			(pintype "passive")
@@
 			(layers "*.Cu" "*.Mask")
 			(remove_unused_layers no)
-			(net 15 "Net-(J1-Pin_4)")
+			(net 14 "Net-(J1-Pin_4)")
 			(pinfunction "GPIO6/SDA")
 			(pintype "passive")
@@
 			(layers "F.Cu" "F.Mask")
 			(roundrect_rratio 0.1)
-			(net 16 "Net-(J1-Pin_3)")
+			(net 15 "Net-(J1-Pin_3)")
 			(pinfunction "GPIO7/SCL")
 			(pintype "passive")
@@
 			(layers "*.Cu" "*.Mask")
 			(remove_unused_layers no)
-			(net 16 "Net-(J1-Pin_3)")
+			(net 15 "Net-(J1-Pin_3)")
 			(pinfunction "GPIO7/SCL")
 			(pintype "passive")
@@
 			(layers "*.Cu" "*.Mask")
 			(remove_unused_layers no)
-			(net 14 "unconnected-(U1-3V3-Pad12)")
+			(net 16 "unconnected-(U1-3V3-Pad12)_1")
 			(pinfunction "3V3")
-			(pintype "passive")
+			(pintype "passive+no_connect")
 		)
 		(pad "12" smd roundrect
@@
 			(layers "F.Cu" "F.Mask")
 			(roundrect_rratio 0.1)
-			(net 14 "unconnected-(U1-3V3-Pad12)")
+			(net 16 "unconnected-(U1-3V3-Pad12)_1")
 			(pinfunction "3V3")
-			(pintype "passive")
+			(pintype "passive+no_connect")
 			(thermal_bridge_angle 45)
 		)
@@
 			(layers "*.Cu" "*.Mask")
 			(remove_unused_layers no)
-			(net 16 "Net-(J1-Pin_3)")
+			(net 15 "Net-(J1-Pin_3)")
 			(pinfunction "Pin_3")
 			(pintype "passive")
@@
 			(layers "*.Cu" "*.Mask")
 			(remove_unused_layers no)
-			(net 15 "Net-(J1-Pin_4)")
+			(net 14 "Net-(J1-Pin_4)")
 			(pinfunction "Pin_4")
 			(pintype "passive")
@@
 			(layers "*.Cu" "*.Mask")
 			(remove_unused_layers no)
-			(net 7 "Net-(U1-GPIO3{slash}MOSI)")
+			(net 3 "GND")
 			(pinfunction "S2")
 			(pintype "passive")
@@
 			(net 5 "unconnected-(D2-DOUT-Pad1)")
 			(pinfunction "DOUT")
-			(pintype "output")
+			(pintype "output+no_connect")
 		)
 		(pad "2" smd rect
@@
 		)
 	)
-	(dimension
-		(type orthogonal)
-		(layer "F.Cu")
-		(pts
-			(xy 147.1 101.0125) (xy 245.96875 59)
-		)
-		(height -42.0125)
-		(orientation 0)
-		(format
-			(prefix "")
-			(suffix "")
-			(units 3)
-			(units_format 0)
-			(precision 4)
-			(suppress_zeroes yes)
-		)
-		(style
-			(thickness 0.2)
-			(arrow_length 1.27)
-			(text_position_mode 0)
-			(arrow_direction outward)
-			(extension_height 0.58642)
-			(extension_offset 0.5)
-			(keep_text_aligned yes)
-		)
-		(gr_text "98.8688"
-			(at 196.534375 57.2 0)
-			(layer "F.Cu")
-			(effects
-				(font
-					(size 1.5 1.5)
-					(thickness 0.3)
-				)
-			)
-		)
-	)
 	(segment
 		(start 242.5775 73.66375)
@@
 	)
 	(segment
+		(start 188.9275 66.91375)
+		(end 186.4275 69.41375)
+		(width 0.2)
+		(layer "F.Cu")
+		(net 3)
+	)
+	(segment
+		(start 186.4275 69.41375)
+		(end 174.4275 69.41375)
+		(width 0.2)
+		(layer "F.Cu")
+		(net 3)
+	)
+	(segment
 		(start 180.975 97.63125)
 		(end 180.975 87.15375)
@@
 	)
 	(segment
-		(start 188.9275 66.91375)
-		(end 182.70575 73.1355)
-		(width 0.2)
-		(layer "F.Cu")
-		(net 7)
-	)
-	(segment
 		(start 164.81844 73.1355)
 		(end 164.19575 72.51281)
@@
 	)
 	(segment
-		(start 182.70575 73.1355)
-		(end 173.20575 73.1355)
-		(width 0.2)
-		(layer "F.Cu")
-		(net 7)
-	)
-	(segment
 		(start 169.26875 72.0725)
 		(end 165.25875 72.0725)
@@
 		(width 0.2)
 		(layer "F.Cu")
-		(net 15)
+		(net 14)
 	)
 	(segment
@@
 		(width 0.2)
 		(layer "F.Cu")
-		(net 15)
+		(net 14)
 	)
 	(segment
@@
 		(width 0.2)
 		(layer "F.Cu")
-		(net 15)
+		(net 14)
 	)
 	(segment
@@
 		(width 0.2)
 		(layer "B.Cu")
-		(net 15)
+		(net 14)
 	)
 	(segment
@@
 		(width 0.2)
 		(layer "F.Cu")
-		(net 16)
+		(net 15)
 	)
 	(segment
@@
 		(width 0.2)
 		(layer "F.Cu")
-		(net 16)
+		(net 15)
 	)
 	(segment
@@
 		(width 0.2)
 		(layer "F.Cu")
-		(net 16)
+		(net 15)
 	)
 	(segment
@@
 		(width 0.2)
 		(layer "F.Cu")
-		(net 16)
+		(net 15)
 	)
 	(segment
@@
 		(width 0.2)
 		(layer "F.Cu")
-		(net 16)
+		(net 15)
 	)
 	(segment
@@
 		(width 0.2)
 		(layer "F.Cu")
-		(net 16)
+		(net 15)
 	)
 	(segment
@@
 		(width 0.2)
 		(layer "F.Cu")
-		(net 16)
+		(net 15)
 	)
 	(segment
@@
 		(width 0.2)
 		(layer "F.Cu")
-		(net 16)
+		(net 15)
 	)
 	(segment
@@
 		(width 0.2)
 		(layer "F.Cu")
-		(net 16)
+		(net 15)
 	)
 	(segment
@@
 		(width 0.2)
 		(layer "F.Cu")
-		(net 16)
+		(net 15)
 	)
 	(segment
@@
 		(width 0.2)
 		(layer "F.Cu")
-		(net 16)
+		(net 15)
 	)
 	(segment
@@
 		(width 0.2)
 		(layer "F.Cu")
-		(net 16)
+		(net 15)
 	)
 	(segment
@@
 		(width 0.2)
 		(layer "F.Cu")
-		(net 16)
+		(net 15)
 	)
 	(segment
@@
 		(width 0.2)
 		(layer "F.Cu")
-		(net 16)
+		(net 15)
 	)
 	(segment
@@
 		(width 0.2)
 		(layer "F.Cu")
-		(net 16)
+		(net 15)
 	)
 	(segment
@@
 		(width 0.2)
 		(layer "F.Cu")
-		(net 16)
+		(net 15)
 	)
 	(segment
@@
 		(width 0.2)
 		(layer "F.Cu")
-		(net 16)
+		(net 15)
 	)
 	(segment
@@
 		(width 0.2)
 		(layer "B.Cu")
-		(net 16)
+		(net 15)
 	)
 	(embedded_fonts no)
