File: PCB/test macropad 1.kicad_sch (KiCad schematic)
At the start: 10 parts, among them J1 Oled Isplay 0.91inch 128x32, SW1 SW_Push, SW2 RotaryEncoder_Switch, SW4 SW_Push, SW6 SW_Push, SW8 SW_Push, SW9 SW_Push, U1 XIAO-RP2040-DIP

Commit message: finally finished
Connections:
- net GND: now also SW2.S2
- net at SW2.B, U1.11 (GPIO3/MOSI): no longer SW2.S2
- no-connect marks 0 -> 2
